File: I2C-LCD-Backpack.brd (EAGLE design)
At the start: 45.7 x 19.1 mm, 22 parts, among them J3 LCD, Q1 MMBT2222A, U1 PCA8574

Commit message: Rev D
Other:
- board text added: "I2C LCD BKPK (D)"
- board text added: "dcity.org"
- board text removed: "I2C LCD BKPK (C)"
- board text removed: "wht.io"
Changed lines of the file:
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@@
 <?xml version="1.0" encoding="utf-8"?>
 <!DOCTYPE eagle SYSTEM "eagle.dtd">
-<eagle version="7.5.0">
+<eagle version="9.1.3">
 <drawing>
 <settings>
 <setting alwaysvectorfont="no"/>
+<setting keepoldvectorfont="yes"/>
 <setting verticaltext="up"/>
 </settings>
@@
 <text x="29.083" y="6.604" size="0.889" layer="21" font="vector" ratio="15" rot="R90">A1</text>
 <text x="31.623" y="6.477" size="0.889" layer="21" font="vector" ratio="15" rot="R90">A2</text>
-<text x="34.798" y="16.002" size="0.889" layer="21" font="vector" ratio="15" rot="R180">I2C LCD BKPK (C)</text>
+<text x="34.798" y="16.002" size="0.889" layer="21" font="vector" ratio="15" rot="R180">I2C LCD BKPK (D)</text>
 <text x="3.175" y="18.161" size="0.889" layer="21" font="vector" ratio="15" rot="R180">Q1</text>
-<text x="40.132" y="14.605" size="0.889" layer="22" font="vector" ratio="15" rot="MR0">I2C LCD BKPK (C)</text>
+<text x="40.132" y="14.605" size="0.889" layer="22" font="vector" ratio="15" rot="MR0">I2C LCD BKPK (D)</text>
 <text x="23.114" y="9.017" size="0.889" layer="21" font="vector" ratio="15" rot="R270">SCL</text>
 <text x="20.574" y="8.89" size="0.889" layer="21" font="vector" ratio="15" rot="R270">SDA</text>
@@
 <rectangle x1="26.797" y1="0.762" x2="27.94" y2="2.667" layer="43"/>
 <rectangle x1="29.337" y1="1.016" x2="30.48" y2="2.794" layer="43"/>
-<text x="22.733" y="12.954" size="1.524" layer="21" font="vector" ratio="10">wht.io</text>
-<text x="36.703" y="12.573" size="1.524" layer="22" font="vector" ratio="10" rot="MR0">wht.io</text>
+<text x="22.733" y="12.954" size="1.524" layer="21" font="vector" ratio="10">dcity.org</text>
+<text x="36.703" y="12.573" size="1.524" layer="22" font="vector" ratio="10" rot="MR0">dcity.org</text>
 </plain>
 <attributes>
@@
 <param name="dpMaxLengthDifference" value="10mm"/>
 <param name="dpGapFactor" value="2.5"/>
-<param name="checkGrid" value="0"/>
 <param name="checkAngle" value="1"/>
 <param name="checkFont" value="1"/>
 <param name="checkRestrict" value="1"/>
+<param name="checkStop" value="0"/>
+<param name="checkValues" value="0"/>
+<param name="checkNames" value="1"/>
+<param name="checkWireStubs" value="1"/>
+<param name="checkPolygonWidth" value="0"/>
 <param name="useDiameter" value="13"/>
 <param name="maxErrors" value="50"/>
@@
 </element>
 <element name="R6" library="0" package="TC33X" value="10K" x="29.845" y="10.795" smashed="yes" rot="R90">
+<attribute name="NAME" x="27.94" y="9.779" size="0.889" layer="25" font="vector" ratio="15" rot="R180"/>
 <attribute name="PROD_ID" value="RES-12428" x="29.845" y="10.795" size="1.778" layer="27" rot="R90" display="off"/>
-<attribute name="NAME" x="27.94" y="9.779" size="0.889" layer="25" font="vector" ratio="15" rot="R180"/>
 </element>
 <element name="Q1" library="0" package="SOT23-3" value="MMBT2222A" x="2.54" y="15.24" smashed="yes" rot="R90">
@@
 </element>
 <element name="U1" library="0" package="TSSOP16" value="PCA8574" x="17.018" y="12.065" smashed="yes" rot="R90">
+<attribute name="NAME" x="14.986" y="8.001" size="0.889" layer="25" font="vector" ratio="15"/>
 <attribute name="VALUE" x="17.653" y="8.001" size="1.27" layer="27" ratio="10" rot="R90"/>
-<attribute name="NAME" x="14.986" y="8.001" size="0.889" layer="25" font="vector" ratio="15"/>
 </element>
 <element name="R7" library="0" package="0805-RES" value="4.7k" x="20.955" y="1.905" smashed="yes" rot="R90">
@@
 </signal>
 </signals>
+<mfgpreviewcolors>
+<mfgpreviewcolor name="soldermaskcolor" color="0xC8008000"/>
+<mfgpreviewcolor name="silkscreencolor" color="0xFFFEFEFE"/>
+<mfgpreviewcolor name="backgroundcolor" color="0xFF282828"/>
+<mfgpreviewcolor name="coppercolor" color="0xFFFFBF00"/>
+<mfgpreviewcolor name="substratecolor" color="0xFF786E46"/>
+</mfgpreviewcolors>
 </board>
 </drawing>

Commit message: Rev E
Parts:
- J1, J2: value (none) -> QWIIC_RIGHT_ANGLE; device 0:HW4-SMD-2.0-90D -> 0:JST04_1MM_RA
- moved J2 5.22 mm to (40.8, 6.73), turned to 90 degrees
- moved J1 5.22 mm to (4.95, 6.73), turned to 270 degrees
Connections:
- net GND: now also J1.1, J2.1; no longer J1.4, J2.4
- net SCL: now also J1.4, J2.4; no longer J1.1, J2.1
- net SDA: now also J1.3, J2.3; no longer J1.2, J2.2
- net VCC: now also J1.2, J2.2; no longer J1.3, J2.3
Routing:
- net VCC: track 102.6 -> 113.1 mm
- net SDA: track 37.1 -> 46.2 mm
- net SCL: track 52.5 -> 54.1 mm, vias 2 -> 3
- net GND: track 18.7 -> 19.4 mm
Other:
- board text added: "GND"
- board text added: "I2C LCD BKPK (E)"
- board text added: "VCC"
- board text removed: "I2C LCD BKPK (D)"
